File: hardware/audio.kicad_sch (KiCad schematic)
At the start: 22 parts, among them J2 Left, J3 Right, U4 AMS1117-3.3, U5 AMS1117-3.3, U6 PCM5102A

Commit message: Finished first iteration of the PCB
Parts:
- removed J2: Left, RCJ-013:CUI_RCJ-013, symbol RCJ-013:RCJ-013
- removed J3: Right, RCJ-013:CUI_RCJ-013, symbol RCJ-013:RCJ-013
- added TP20: AVDD, TestPoint:TestPoint_Pad_D1.0mm, symbol Connector:TestPoint
- added TP21: CPVDD, TestPoint:TestPoint_Pad_D1.0mm, symbol Connector:TestPoint
- R21: renamed from R10; LCSC# (none) -> C25117; LSCS# C25117 -> (none)
- R22: renamed from R11; LCSC# (none) -> C25117; LSCS# C25117 -> (none)
- U6: renamed from U4; LCSC# (none) -> C6186; LSCS# C6186 -> (none)
- U7: renamed from U5; LCSC# (none) -> C6186; LSCS# C6186 -> (none)
- gave numbers to parts that had none: 1
- renumbered C7 to C12, C8 to C13, C9 to C14, C10 to C15, C11 to C16, C12 to C17, C13 to C18, C14 to C19, C15 to C20, C16 to C21, C17 to C22, C18 to C23, C19 to C24, C20 to C25, U6 to U8
Connections:
- net AVVD is gone; now on net AVDD: U6.2 (VO)
- net AVDD: now also TP20.1
- net CPVDD: now also TP21.1
- net GND: now also C20.1
- net OUT_L: now also C24.2, R21.1; no longer R21.2
- net OUT_R: now also C25.2
- net MUTE: now reaches U8.17 (XSMT)
- net at R22.1, U8.7 (OUTR): no longer C25.2
- new net: R21.2, U8.6 (OUTL)
Other:
- note removed: "Output"
- moved on the sheet: R21, R22
