File: hardware/input.kicad_sch (KiCad schematic)
At the start: 10 parts, among them Q1 AO3400A, Q2 AO3401A

Commit message: Fixed flipped transistor
Connections:
- net Vin: now also Q2.3 (D); no longer Q2.2 (S)
- net at D1.1 (K), R5.1: now also Q2.2 (S); no longer Q2.3 (D)
Changed lines of the file:
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@@
     (pin "2")
   )
-  (symbol (lib_id "Transistor_FET:AO3401A") (at 82.55 58.42 0) (unit 1)
+  (symbol (lib_id "Transistor_FET:AO3401A") (at 82.55 58.42 0) (mirror x) (unit 1)
     (in_bom yes) (on_board yes) (fields_autoplaced)
     (property "Reference" "Q2" (id 0) (at 87.757 57.5853 0)
@@
       (effects (font (size 1.27 1.27)) (justify left))
     )
-    (property "Footprint" "Package_TO_SOT_SMD:SOT-23" (id 2) (at 87.63 60.325 0)
+    (property "Footprint" "Package_TO_SOT_SMD:SOT-23" (id 2) (at 87.63 56.515 0)
       (effects (font (size 1.27 1.27) italic) (justify left) hide)
     )

Commit message: Finished first iteration of the PCB
Parts:
- removed D2: 1N5819WS, Diode_SMD:D_SOD-323, symbol Device:D_Schottky
- removed R6: 20k, Resistor_SMD:R_0402_1005Metric, symbol Device:R
- removed R7: 10k, Resistor_SMD:R_0402_1005Metric, symbol Device:R
- added C10: 22u, Capacitor_SMD:C_1206_3216Metric, symbol Device:C
- added D3: 1N5819WS, Diode_SMD:D_SOD-323, symbol Device:D_Schottky
- added R16: 1k, Resistor_SMD:R_0402_1005Metric, symbol Device:R
- renumbered D1 to D4, Q1 to Q3, Q2 to Q4, R4 to R17, R5 to R18, R8 to R19, R9 to R20
Connections:
- net GND: now also C10.2
- net +12V renamed Dashboard Light
- net Dashboard Light: now also D3.2 (A)
- net +BATT renamed Car Battery
- net POWER_CONTROL: no longer names the net of Q3.1 (G), R17.1
- net POWER_CONTROL: now also C10.1, R16.1
- net SUPPLY_SENSE renamed Sense
- net Vin renamed V_in
- new net: D3.1 (K), R16.2
Other:
- moved on the sheet: D4, Q3, Q4, R17, R18, R19, R20
